File: PCB/KEYBOARD75.kicad_pcb (KiCad board)
At the start: 2 copper layers, 315.9 x 124.1 mm, 367 parts, among them J1 USB_C_Receptacle_USB2.0_16P, SW1 ESC, SW10 F9, SW11 F10, SW12 F11, SW13 F12, SW14 Delete, SW15 `, SW16 1, SW17 2, SW18 3, SW19 4, SW2 F1, SW20 5, SW21 6, SW22 7, SW23 8, SW24 9, SW25 0, SW26 -, SW27 +, SW28 Backspace, SW29 Home, SW3 F2, SW30 Tab, SW31 Q, SW32 W, SW33 E, SW34 R, SW35 T, SW36 Y, SW37 U, SW38 I, SW39 O, SW4 F3, SW40 P, SW41 [, SW42 ], SW43 \, SW44 Pg Up, SW45 Caps Lock, SW46 A, SW47 S, SW48 D, SW49 F, SW5 F4, SW50 G, SW51 H, SW52 J, SW53 K, SW54 L, SW55 ;, SW56 ", SW57 Enter, SW58 Pg Dn, SW59 L Shift, SW6 F5, SW60 Z, SW61 X, SW62 C, SW63 V, SW64 B, SW65 N, SW66 M, SW67 ,, SW68 ., SW69 /, SW7 F6, SW70 R Shift, SW71 Up Arrow, SW72 End, SW73 L Ctrl, SW74 Win, SW75 Alt, SW76 Space, SW77 Alt, SW78 Fn, SW79 R Ctrl, SW8 F7, SW80 Left Arrow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

Commit message: Add files via upload
Parts:
- turned C97 to 0 degrees
- turned C98 to 180 degrees
Connections:
- C97 pad 1: +3.3V -> GND
- C97 pad 2: GND -> +3.3V
- C98 pad 1: +3.3V -> GND
- C98 pad 2: GND -> +3.3V
- U1 pad 43: GND -> +3.3V
- U1 pad 44: GND -> +3.3V
- U1 pad 48: GND -> +3.3V
Routing:
- net GND: track 626.7 -> 623.3 mm, vias 93 -> 94
- net +3.3V: track 57.4 -> 59.5 mm
